File: builds/gx140/gx140_rev2.kicad_sch (KiCad schematic)
At the start: 14 parts, among them M1 Specter_1804_FL_CCW, M2 Specter_1804_FR_CW, M3 Specter_1804_RL_CCW, M4 Specter_1804_RR_CW

Commit message: Reverse wire tag all net labels in KiCad schematic
Rename all signal net labels to encode source-to-destination path:
  DSHOT_M1  -> FC_M1_TO_ESC_S1
  CAM_VIDEO -> CAM_VID_TO_FC_VIN
  VTX_VIDEO -> FC_VOUT_TO_VTX_VID
  TX4_SMARTAUDIO -> FC_TX4_TO_VTX_SA
  TX5_CRSF  -> FC_TX5_TO_RX_CRSF
  RX5_CRSF  -> FC_RX5_FROM_RX_CRSF
  TX3_GPS   -> FC_TX3_TO_GPS_RX
  RX3_GPS   -> FC_RX3_FROM_GPS_TX
  ESC_CURR  -> ESC_CURR_TO_FC

Every net label now reads as a reverse wire tag — at the
destination pin you see exactly where the signal came from.

Co-Authored-By: Claude Sonnet 4.6 (1M context) <noreply@anthropic.com>
Connections:
- net CAM_VIDEO renamed CAM_VID_TO_FC_VIN
- net DSHOT_M1 renamed FC_M1_TO_ESC_S1
- net DSHOT_M2 renamed FC_M2_TO_ESC_S2
- net DSHOT_M3 renamed FC_M3_TO_ESC_S3
- net DSHOT_M4 renamed FC_M4_TO_ESC_S4
- net ESC_CURR renamed ESC_CURR_TO_FC
- net RX3_GPS renamed FC_RX3_FROM_GPS_TX
- net RX5_CRSF renamed FC_RX5_FROM_RX_CRSF
- net TX3_GPS renamed FC_TX3_TO_GPS_RX
- net TX4_SMARTAUDIO renamed FC_TX4_TO_VTX_SA
- net TX5_CRSF renamed FC_TX5_TO_RX_CRSF
- net VTX_VIDEO renamed FC_VOUT_TO_VTX_VID
Changed lines of the file:
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@@
     (effects (font (size 1.27 1.27)) (justify right))
   )
-  (label "DSHOT_M1" (at 93.98 83.82 0)
+  (label "FC_M1_TO_ESC_S1" (at 93.98 83.82 0)
     (effects (font (size 1.27 1.27)) (justify right))
   )
-  (label "DSHOT_M2" (at 93.98 86.36 0)
+  (label "FC_M2_TO_ESC_S2" (at 93.98 86.36 0)
     (effects (font (size 1.27 1.27)) (justify right))
   )
-  (label "DSHOT_M3" (at 93.98 88.9 0)
+  (label "FC_M3_TO_ESC_S3" (at 93.98 88.9 0)
     (effects (font (size 1.27 1.27)) (justify right))
   )
-  (label "DSHOT_M4" (at 93.98 91.44 0)
+  (label "FC_M4_TO_ESC_S4" (at 93.98 91.44 0)
     (effects (font (size 1.27 1.27)) (justify right))
   )
-  (label "ESC_CURR" (at 93.98 93.98 0)
+  (label "ESC_CURR_TO_FC" (at 93.98 93.98 0)
     (effects (font (size 1.27 1.27)) (justify right))
   )
@@
     (effects (font (size 1.27 1.27)) (justify right))
   )
-  (label "ESC_CURR" (at 93.98 167.64 0)
+  (label "ESC_CURR_TO_FC" (at 93.98 167.64 0)
     (effects (font (size 1.27 1.27)) (justify right))
   )
-  (label "DSHOT_M1" (at 93.98 170.18 0)
+  (label "FC_M1_TO_ESC_S1" (at 93.98 170.18 0)
     (effects (font (size 1.27 1.27)) (justify right))
   )
-  (label "DSHOT_M2" (at 93.98 172.72 0)
+  (label "FC_M2_TO_ESC_S2" (at 93.98 172.72 0)
     (effects (font (size 1.27 1.27)) (justify right))
   )
-  (label "DSHOT_M3" (at 93.98 175.26 0)
+  (label "FC_M3_TO_ESC_S3" (at 93.98 175.26 0)
     (effects (font (size 1.27 1.27)) (justify right))
   )
-  (label "DSHOT_M4" (at 93.98 177.8 0)
+  (label "FC_M4_TO_ESC_S4" (at 93.98 177.8 0)
     (effects (font (size 1.27 1.27)) (justify right))
   )
@@
     (effects (font (size 1.27 1.27)) (justify left))
   )
-  (label "CAM_VIDEO" (at 160.02 165.1 0)
+  (label "CAM_VID_TO_FC_VIN" (at 160.02 165.1 0)
     (effects (font (size 1.27 1.27)) (justify left))
   )
-  (label "VTX_VIDEO" (at 160.02 167.64 0)
+  (label "FC_VOUT_TO_VTX_VID" (at 160.02 167.64 0)
     (effects (font (size 1.27 1.27)) (justify left))
   )
-  (label "TX4_SMARTAUDIO" (at 160.02 170.18 0)
+  (label "FC_TX4_TO_VTX_SA" (at 160.02 170.18 0)
     (effects (font (size 1.27 1.27)) (justify left))
   )
-  (label "TX5_CRSF" (at 160.02 175.26 0)
+  (label "FC_TX5_TO_RX_CRSF" (at 160.02 175.26 0)
     (effects (font (size 1.27 1.27)) (justify left))
   )
-  (label "RX5_CRSF" (at 160.02 177.8 0)
+  (label "FC_RX5_FROM_RX_CRSF" (at 160.02 177.8 0)
     (effects (font (size 1.27 1.27)) (justify left))
   )
-  (label "TX3_GPS" (at 160.02 180.34 0)
+  (label "FC_TX3_TO_GPS_RX" (at 160.02 180.34 0)
     (effects (font (size 1.27 1.27)) (justify left))
   )
-  (label "RX3_GPS" (at 160.02 182.88 0)
+  (label "FC_RX3_FROM_GPS_TX" (at 160.02 182.88 0)
     (effects (font (size 1.27 1.27)) (justify left))
   )
@@
     (effects (font (size 1.27 1.27)) (justify right))
   )
-  (label "VTX_VIDEO" (at 254.0 148.59 0)
+  (label "FC_VOUT_TO_VTX_VID" (at 254.0 148.59 0)
     (effects (font (size 1.27 1.27)) (justify right))
   )
-  (label "TX4_SMARTAUDIO" (at 254.0 151.13 0)
+  (label "FC_TX4_TO_VTX_SA" (at 254.0 151.13 0)
     (effects (font (size 1.27 1.27)) (justify right))
   )
@@
     (effects (font (size 1.27 1.27)) (justify right))
   )
-  (label "CAM_VIDEO" (at 307.34 173.99 0)
+  (label "CAM_VID_TO_FC_VIN" (at 307.34 173.99 0)
     (effects (font (size 1.27 1.27)) (justify left))
   )
@@
     (effects (font (size 1.27 1.27)) (justify right))
   )
-  (label "TX5_CRSF" (at 254.0 199.39 0)
+  (label "FC_TX5_TO_RX_CRSF" (at 254.0 199.39 0)
     (effects (font (size 1.27 1.27)) (justify right))
   )
-  (label "RX5_CRSF" (at 254.0 201.93 0)
+  (label "FC_RX5_FROM_RX_CRSF" (at 254.0 201.93 0)
     (effects (font (size 1.27 1.27)) (justify right))
   )
@@
     (effects (font (size 1.27 1.27)) (justify right))
   )
-  (label "TX3_GPS" (at 254.0 229.87 0)
+  (label "FC_TX3_TO_GPS_RX" (at 254.0 229.87 0)
     (effects (font (size 1.27 1.27)) (justify right))
   )
-  (label "RX3_GPS" (at 254.0 232.41 0)
+  (label "FC_RX3_FROM_GPS_TX" (at 254.0 232.41 0)
     (effects (font (size 1.27 1.27)) (justify right))
   )
